File: MOS6566_Adapter.kicad_sch (KiCad schematic)
At the start: 12 parts, among them U1 MOS6566, U2 MOS6567/MOS8562, U3 74HCT04, U4 74HCT245, U5 74HCT573, U6 74HCT573

Commit message: Finetuning
Parts:
- added C5: C_Small, Custom_Caps:C_Disc_D3.4mm_W2.1mm_P2.50mm, symbol Device:C_Small
Connections:
- net GND: now also C5.2
- net PwR5V: now also C5.1
Other:
- moved on the sheet: C1, C2, C3, C4
Changed lines of the file:
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@@
 	)
 	(label "PwR5V"
-		(at 113.03 172.72 0)
+		(at 104.14 172.72 0)
 		(fields_autoplaced yes)
 		(effects
@@
 		)
 	)
+	(label "GND"
+		(at 163.83 177.8 270)
+		(fields_autoplaced yes)
+		(effects
+			(font
+				(size 1.27 1.27)
+			)
+			(justify right bottom)
+		)
+	)
 	(label "D2"
 		(at 46.99 62.23 180)
@@
 	)
 	(label "PwR5V"
-		(at 127 172.72 0)
+		(at 163.83 172.72 0)
+		(fields_autoplaced yes)
+		(effects
+			(font
+				(size 1.27 1.27)
+			)
+			(justify left bottom)
+		)
+	)
+	(label "PwR5V"
+		(at 118.11 172.72 0)
 		(fields_autoplaced yes)
 		(effects
@@
 	)
 	(label "GND"
-		(at 113.03 177.8 270)
+		(at 104.14 177.8 270)
 		(fields_autoplaced yes)
 		(effects
@@
 	)
 	(label "GND"
-		(at 142.24 177.8 270)
+		(at 133.35 177.8 270)
 		(fields_autoplaced yes)
 		(effects
@@
 	)
 	(label "GND"
-		(at 156.21 177.8 270)
+		(at 147.32 177.8 270)
 		(fields_autoplaced yes)
 		(effects
@@
 	)
 	(label "PwR5V"
-		(at 156.21 172.72 0)
+		(at 147.32 172.72 0)
 		(fields_autoplaced yes)
 		(effects
@@
 	)
 	(label "GND"
-		(at 127 177.8 270)
+		(at 118.11 177.8 270)
 		(fields_autoplaced yes)
 		(effects
@@
 	)
 	(label "PwR5V"
-		(at 142.24 172.72 0)
+		(at 133.35 172.72 0)
 		(fields_autoplaced yes)
 		(effects
@@
 	(symbol
 		(lib_id "Device:C_Small")
-		(at 127 175.26 0)
+		(at 118.11 175.26 0)
 		(unit 1)
 		(exclude_from_sim no)
@@
 		(fields_autoplaced yes)
 		(property "Reference" "C2"
-			(at 129.54 173.9962 0)
+			(at 120.65 173.9962 0)
 			(effects
 				(font
@@
 		)
 		(property "Value" "C_Small"
-			(at 129.54 176.5362 0)
+			(at 120.65 176.5362 0)
 			(effects
 				(font
@@
 		)
 		(property "Footprint" "Custom_Caps:C_Disc_D3.4mm_W2.1mm_P2.50mm"
-			(at 127 175.26 0)
+			(at 118.11 175.26 0)
 			(effects
 				(font
@@
 		)
 		(property "Datasheet" "~"
-			(at 127 175.26 0)
+			(at 118.11 175.26 0)
 			(effects
 				(font
@@
 		)
 		(property "Description" "Unpolarized capacitor, small symbol"
-			(at 127 175.26 0)
+			(at 118.11 175.26 0)
 			(effects
 				(font
@@
 	(symbol
 		(lib_id "Device:C_Small")
-		(at 113.03 175.26 0)
+		(at 104.14 175.26 0)
 		(unit 1)
 		(exclude_from_sim no)
@@
 		(fields_autoplaced yes)
 		(property "Reference" "C1"
-			(at 115.57 173.9962 0)
+			(at 106.68 173.9962 0)
 			(effects
 				(font
@@
 		)
 		(property "Value" "C_Small"
-			(at 115.57 176.5362 0)
+			(at 106.68 176.5362 0)
 			(effects
 				(font
@@
 		)
 		(property "Footprint" "Custom_Caps:C_Disc_D3.4mm_W2.1mm_P2.50mm"
-			(at 113.03 175.26 0)
+			(at 104.14 175.26 0)
 			(effects
 				(font
@@
 		)
 		(property "Datasheet" "~"
-			(at 113.03 175.26 0)
+			(at 104.14 175.26 0)
 			(effects
 				(font
@@
 		)
 		(property "Description" "Unpolarized capacitor, small symbol"
-			(at 113.03 175.26 0)
+			(at 104.14 175.26 0)
 			(effects
 				(font
@@
 		(dnp no)
 		(property "Reference" "U3"
-			(at 133.35 183.642 90)
+			(at 133.35 186.69 90)
 			(effects
 				(font
@@
 	(symbol
 		(lib_id "Device:C_Small")
-		(at 142.24 175.26 0)
+		(at 133.35 175.26 0)
 		(unit 1)
 		(exclude_from_sim no)
@@
 		(fields_autoplaced yes)
 		(property "Reference" "C3"
-			(at 144.78 173.9962 0)
+			(at 135.89 173.9962 0)
 			(effects
 				(font
@@
 		)
 		(property "Value" "C_Small"
-			(at 144.78 176.5362 0)
+			(at 135.89 176.5362 0)
 			(effects
 				(font
@@
 		)
 		(property "Footprint" "Custom_Caps:C_Disc_D3.4mm_W2.1mm_P2.50mm"
-			(at 142.24 175.26 0)
+			(at 133.35 175.26 0)
 			(effects
 				(font
@@
 		)
 		(property "Datasheet" "~"
-			(at 142.24 175.26 0)
+			(at 133.35 175.26 0)
 			(effects
 				(font
@@
 		)
 		(property "Description" "Unpolarized capacitor, small symbol"
-			(at 142.24 175.26 0)
+			(at 133.35 175.26 0)
 			(effects
 				(font
@@
 	(symbol
 		(lib_id "Device:C_Small")
-		(at 156.21 175.26 0)
+		(at 163.83 175.26 0)
 		(unit 1)
 		(exclude_from_sim no)
@@
 		(dnp no)
 		(fields_autoplaced yes)
+		(property "Reference" "C5"
+			(at 166.37 173.9962 0)
+			(effects
+				(font
+					(size 1.27 1.27)
+				)
+				(justify left)
+			)
+		)
+		(property "Value" "C_Small"
+			(at 166.37 176.5362 0)
+			(effects
+				(font
+					(size 1.27 1.27)
+				)
+				(justify left)
+			)
+		)
+		(property "Footprint" "Custom_Caps:C_Disc_D3.4mm_W2.1mm_P2.50mm"
+			(at 163.83 175.26 0)
+			(effects
+				(font
+					(size 1.27 1.27)
+				)
+				(hide yes)
+			)
+		)
+		(property "Datasheet" "~"
+			(at 163.83 175.26 0)
+			(effects
+				(font
+					(size 1.27 1.27)
+				)
+				(hide yes)
+			)
+		)
+		(property "Description" "Unpolarized capacitor, small symbol"
+			(at 163.83 175.26 0)
+			(effects
+				(font
+					(size 1.27 1.27)
+				)
+				(hide yes)
+			)
+		)
+		(pin "1"
+		)
+		(pin "2"
+		)
+		(instances
+			(project "MOS6566_Adapter"
+				(path "/a1e026d0-e5d1-47a2-a430-e4a7fc52c075"
+					(reference "C5")
+					(unit 1)
+				)
+			)
+		)
+	)
+	(symbol
+		(lib_id "Device:C_Small")
+		(at 147.32 175.26 0)
+		(unit 1)
+		(exclude_from_sim no)
+		(in_bom yes)
+		(on_board yes)
+		(dnp no)
+		(fields_autoplaced yes)
 		(property "Reference" "C4"
-			(at 158.75 173.9962 0)
+			(at 149.86 173.9962 0)
 			(effects
 				(font
@@
 		)
 		(property "Value" "C_Small"
-			(at 158.75 176.5362 0)
+			(at 149.86 176.5362 0)
 			(effects
 				(font
@@
 		)
 		(property "Footprint" "Custom_Caps:C_Disc_D3.4mm_W2.1mm_P2.50mm"
-			(at 156.21 175.26 0)
+			(at 147.32 175.26 0)
 			(effects
 				(font
@@
 		)
 		(property "Datasheet" "~"
-			(at 156.21 175.26 0)
+			(at 147.32 175.26 0)
 			(effects
 				(font
@@
 		)
 		(property "Description" "Unpolarized capacitor, small symbol"
-			(at 156.21 175.26 0)
-			(effects
-				(font
+			(at 147.32 175.26 0)
+			(effects
+				(font

Commit message: Minor cosmetics
Parts:
- U1, U2: footprint Package_DIP:DIP-40_W15.24mm -> Package_DIP:DIP-40_W15.24mm_Socket
Changed lines of the file:
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@@
 			)
 		)
-		(property "Footprint" "Package_DIP:DIP-40_W15.24mm"
+		(property "Footprint" "Package_DIP:DIP-40_W15.24mm_Socket"
 			(at 59.69 39.37 0)
 			(effects
@@
 			)
 		)
-		(property "Footprint" "Package_DIP:DIP-40_W15.24mm"
+		(property "Footprint" "Package_DIP:DIP-40_W15.24mm_Socket"
 			(at 243.84 40.64 0)
 			(effects
